File: hw/kicad/v4.0/fb.sch (KiCad schematic (older format))
At the start: 48 parts, among them J1 RJ45_LED, U15 SN65176B, U16 SN65176B, U19 SN65176B, U7 LM358

Commit message: Version for ST IGBT Modules
Connections:
- wire segments 227 -> 234
Changed lines of the file:
@@
 Wire Wire Line
 	3500 5000 3500 6150
+Wire Wire Line
+	2750 3000 5200 3000
+Wire Wire Line
+	5200 3000 5200 4100
+Wire Wire Line
+	4900 4800 4900 5000
+Wire Wire Line
+	4900 5000 6100 5000
+Connection ~ 6100 5000
+Wire Wire Line
+	4900 5100 5250 5100
+Wire Wire Line
+	5250 5100 5250 4200
+Wire Wire Line
+	5250 4200 4900 4200
+Connection ~ 4900 5100
 $EndSCHEMATC
