File: hw/kicad/v4.0/f3.sch (KiCad schematic (older format))
At the start: 34 parts, among them P11 USB_OTG, P12 CONN_01X04, P7 CONN_01X04, T1 testpoint, T2 testpoint, T44 testpoint, T45 testpoint, T46 testpoint, U21 USBLC6-4SC6, U25 STM32F303CBTx, U29 USBLC6-4SC6, Y1 8M

Commit message: Version for ST IGBT Modules
Connections:
- net labels added: USB_N, USB_P
- net labels removed: USB_DM, USB_DP
Changed lines of the file:
@@
 $EndComp
 Text HLabel 10500 4000 2    60   Input ~ 0
-USB_DP
+USB_P
 Text HLabel 10500 3900 2    60   Input ~ 0
-USB_DM
+USB_N
 Text HLabel 11000 4400 2    60   Input ~ 0
 HV_EN
@@
 SWCLK
 Text HLabel 3200 5750 0    60   Input ~ 0
-USB_DP
+USB_P
 Text HLabel 3200 5550 0    60   Input ~ 0
-USB_DM
+USB_N
 Text HLabel 5500 5550 2    60   Input ~ 0
 IO_TX
@@
 	7300 5050 7300 5150
 Text HLabel 7800 5550 2    60   Input ~ 0
-USB_DM
+USB_N
 Wire Wire Line
 	7800 5550 7700 5550
 Text HLabel 7800 5650 2    60   Input ~ 0
-USB_DP
+USB_P
 Wire Wire Line
 	7800 5650 7700 5650

Commit message: changed orientation of IGBT module, other improvements
* removed USB port
* better power distribution for F3
Parts:
- removed P11: USB_OTG, stmbl:USB_Micro-B, symbol stmbl:USB_OTG
- removed R150: 1.5k, stmbl:R_0603, symbol stmbl:R
- removed R151, R152: 22, stmbl:R_0603, symbol stmbl:R
- removed T1, T2, T44, T45, T46: testpoint, stmbl:Measurement_Point_Round-SMD-Pad_Small, symbol stmbl:testpoint
Connections:
- net labels removed: USB_N, USB_P
- wire segments 149 -> 144
- no-connect marks 3 -> 1
