File: hw/kicad/v4.0/hv_drive.sch (KiCad schematic (older format))
At the start: 21 parts, among them P6 CONN_01X02, P8 CONN_01X03, U12 IRAM256a

Commit message: Version for ST IGBT Modules
Parts:
- removed C22: 270µ, stmbl:C_Radial_D26_L45_P10, symbol stmbl:CP
- removed U12: IRAM256a, stmbl:IRAM256, symbol stmbl:IRAM256a
- added C146: 100n, stmbl:C_0603, symbol stmbl:C
- added U12: STGIBxx, stmbl:SDIP2B-26L, symbol stgib:STGIBxx
- C21: value 270µ -> 560µ; footprint stmbl:C_Radial_D26_L45_P10 -> Capacitor_THT:CP_Radial_D30.0mm_P10.00mm_SnapIn; Manufacturer No ESMR401VSN271MQ30S -> ESMR401VSN561MA30S
- C42, C43, C44: value 2.2µ -> 3.3µ
Connections:
- wire segments 78 -> 74

Commit message: changed orientation of IGBT module, other improvements
* removed USB port
* better power distribution for F3
Parts:
- added C22: 270µ, Capacitor_THT:CP_Radial_D26.0mm_P10.00mm_SnapIn, symbol stmbl:CP
- C21: value 560µ -> 270µ; footprint Capacitor_THT:CP_Radial_D30.0mm_P10.00mm_SnapIn -> Capacitor_THT:CP_Radial_D26.0mm_P10.00mm_SnapIn
Connections:
- wire segments 74 -> 76
Changed lines of the file:
@@
 P 1600 2600
 F 0 "C21" H 1625 2700 50  0000 L CNN
-F 1 "560µ" H 1625 2500 50  0000 L CNN
-F 2 "Capacitor_THT:CP_Radial_D30.0mm_P10.00mm_SnapIn" H 1638 2450 30  0001 C CNN
+F 1 "270µ" H 1625 2500 50  0000 L CNN
+F 2 "Capacitor_THT:CP_Radial_D26.0mm_P10.00mm_SnapIn" H 1638 2450 30  0001 C CNN
 F 3 "" H 1600 2600 60  0000 C CNN
 F 4 "ESMR401VSN561MA30S" H 1600 2600 60  0001 C CNN "Manufacturer No"
@@
 F 10 "Phoenix" H -2850 -800 50  0001 C CNN "Manufacturer"
 	1    1050 1150
-	-1   0    0    -1
+	-1   0    0    1
 $EndComp
 $Comp
@@
 Connection ~ 10250 3450
 Wire Wire Line
-	1600 2450 2200 2450
-Wire Wire Line
-	1600 2750 2200 2750
+	1600 2450 1900 2450
+Wire Wire Line
+	1600 2750 1900 2750
+$Comp
+L stmbl:CP C22
+U 1 1 5B899BC1
+P 1900 2600
+F 0 "C22" H 1925 2700 50  0000 L CNN
+F 1 "270µ" H 1925 2500 50  0000 L CNN
+F 2 "Capacitor_THT:CP_Radial_D26.0mm_P10.00mm_SnapIn" H 1938 2450 30  0001 C CNN
+F 3 "" H 1900 2600 60  0000 C CNN
+F 4 "ESMR401VSN561MA30S" H 1900 2600 60  0001 C CNN "Manufacturer No"
+F 5 "400V" H 1900 2600 60  0001 C CNN "Voltage"
+F 6 "United Chemi-Con" H -1150 -1800 50  0001 C CNN "Manufacturer"
+	1    1900 2600
+	1    0    0    -1
+$EndComp
+Connection ~ 1900 2450
+Wire Wire Line
+	1900 2450 2200 2450
+Connection ~ 1900 2750
+Wire Wire Line
+	1900 2750 2200 2750
 $EndSCHEMATC
